File: ESProg/ESProg.kicad_pcb (KiCad board)
At the start: 2 copper layers, 45 x 64.2 mm, 6 parts, among them J1 

Commit message: Update with Hackster logo
Parts:
- added  : , alexglow-footprints:hlogoTiny, B.Cu at (140.5, 85.5)
Other:
- board text added: "bit.ly/ouija8266"
Changed lines of the file:
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@@
   (general
     (thickness 1.6)
-    (drawings 55)
+    (drawings 56)
     (tracks 39)
     (zones 0)
-    (modules 6)
+    (modules 7)
     (nets 10)
   )
@@
     (35 F.Paste user)
     (36 B.SilkS user)
-    (37 F.SilkS user hide)
+    (37 F.SilkS user)
     (38 B.Mask user)
     (39 F.Mask user)
@@
     (add_net "Net-(U1-Pad7)")
   )
+  (module alexglow-footprints:hlogoTiny (layer B.Cu)
+    (at 140.5 85.5)
+    (fp_text reference " " (at 0 0) (layer B.SilkS) hide
+      (effects (font (size 1.524 1.524) (thickness 0.3)) (justify mirror))
+    )
+    (fp_text value " " (at 0.75 0) (layer B.SilkS) hide
+      (effects (font (size 1.524 1.524) (thickness 0.3)) (justify mirror))
+    )
+    (fp_poly (pts (xy 0.96307 3.698113) (xy 1.600978 3.489318) (xy 2.182032 3.178598) (xy 2.69637 2.775715)
+      (xy 3.134135 2.290431) (xy 3.485466 1.732507) (xy 3.740505 1.111707) (xy 3.889393 0.437792)
+      (xy 3.91433 0.194914) (xy 3.898804 -0.440859) (xy 3.765829 -1.070276) (xy 3.524451 -1.675618)
+      (xy 3.183711 -2.239169) (xy 2.752655 -2.74321) (xy 2.240323 -3.170025) (xy 2.17371 -3.215279)
+      (xy 1.649073 -3.495858) (xy 1.054974 -3.697845) (xy 0.427584 -3.813151) (xy -0.196925 -3.833688)
+      (xy -0.478527 -3.808387) (xy -1.145466 -3.658181) (xy -1.76114 -3.399154) (xy -2.315181 -3.04246)
+      (xy -2.797226 -2.599249) (xy -3.196906 -2.080674) (xy -3.503857 -1.497885) (xy -3.586268 -1.240831)
+      (xy -1.3335 -1.240831) (xy -1.327858 -1.566507) (xy -1.308084 -1.782011) (xy -1.26991 -1.903784)
+      (xy -1.209067 -1.948271) (xy -1.151356 -1.942421) (xy -1.027018 -1.908362) (xy -0.841359 -1.859298)
+      (xy -0.775533 -1.842201) (xy -0.503316 -1.771843) (xy -0.520282 -1.227666) (xy 0.5715 -1.227666)
+      (xy 0.600035 -1.390403) (xy 0.687652 -1.442385) (xy 0.758683 -1.426277) (xy 0.892057 -1.386678)
+      (xy 1.04775 -1.351867) (xy 1.253105 -1.28745) (xy 1.375135 -1.196004) (xy 1.397 -1.135224)
+      (xy 1.339082 -1.106846) (xy 1.187544 -1.086776) (xy 0.98425 -1.0795) (xy 0.76212 -1.082617)
+      (xy 0.638367 -1.098811) (xy 0.584401 -1.138346) (xy 0.57163 -1.211485) (xy 0.5715 -1.227666)
+      (xy -0.520282 -1.227666) (xy -0.521533 -1.187546) (xy -0.53975 -0.60325) (xy -0.846309 -0.583694)
+      (xy -1.060921 -0.58099) (xy -1.20167 -0.619346) (xy -1.283819 -0.719348) (xy -1.322631 -0.901582)
+      (xy -1.333368 -1.186635) (xy -1.3335 -1.240831) (xy -3.586268 -1.240831) (xy -3.707712 -0.862034)
+      (xy -3.795264 -0.240277) (xy -3.795472 0.315711) (xy -3.787801 0.367228) (xy -2.2225 0.367228)
+      (xy -2.164373 0.342718) (xy -2.011402 0.324958) (xy -1.795706 0.31754) (xy -1.778 0.3175)
+      (xy -1.516426 0.308554) (xy -1.370037 0.280463) (xy -1.32803 0.238125) (xy -1.321467 0.123545)
+      (xy -1.312876 -0.048198) (xy -1.312155 -0.0635) (xy -1.30175 -0.28575) (xy 0.53975 -0.34925)
+      (xy 0.559276 -0.619125) (xy 0.584913 -0.784031) (xy 0.626284 -0.879493) (xy 0.644132 -0.889)
+      (xy 0.732795 -0.872874) (xy 0.909176 -0.830125) (xy 1.138927 -0.769189) (xy 1.196106 -0.753379)
+      (xy 1.48512 -0.673074) (xy 1.778253 -0.592012) (xy 2.01285 -0.527518) (xy 2.016125 -0.526623)
+      (xy 2.200326 -0.466378) (xy 2.321399 -0.407816) (xy 2.3495 -0.376494) (xy 2.291214 -0.348204)
+      (xy 2.137116 -0.32732) (xy 1.918344 -0.317728) (xy 1.876729 -0.3175) (xy 1.403958 -0.3175)
+      (xy 1.36525 0.28575) (xy -0.47625 0.34925) (xy -0.508 0.609254) (xy -0.53975 0.869257)
+      (xy -1.381125 0.643106) (xy -1.686833 0.557519) (xy -1.942925 0.479312) (xy -2.127131 0.415788)
+      (xy -2.217177 0.37425) (xy -2.2225 0.367228) (xy -3.787801 0.367228) (xy -3.720224 0.821045)
+      (xy -3.632552 1.09612) (xy -1.309525 1.09612) (xy -1.210846 1.044669) (xy -0.990353 1.018056)
+      (xy -0.885253 1.016) (xy -0.67566 1.018568) (xy -0.562984 1.036397) (xy -0.517143 1.084678)
+      (xy -0.515325 1.103475) (xy 0.5715 1.103475) (xy 0.5715 0.5715) (xy 1.397 0.5715)
+      (xy 1.397 1.23825) (xy 1.393862 1.511962) (xy 1.385378 1.731219) (xy 1.372939 1.86979)
+      (xy 1.361619 1.905) (xy 1.242834 1.886719) (xy 1.061954 1.841553) (xy 0.868727 1.784021)
+      (xy 0.712898 1.728645) (xy 0.650875 1.69756) (xy 0.604402 1.591472) (xy 0.577918 1.364094)
+      (xy 0.5715 1.103475) (xy -0.515325 1.103475) (xy -0.508055 1.178601) (xy -0.508 1.2065)
+      (xy -0.509841 1.321659) (xy -0.534892 1.377726) (xy -0.612444 1.384062) (xy -0.77179 1.350028)
+      (xy -0.876756 1.324336) (xy -1.142273 1.24347) (xy -1.286599 1.164892) (xy -1.309525 1.09612)
+      (xy -3.632552 1.09612) (xy -3.559715 1.324646) (xy -3.416173 1.651) (xy -3.255506 1.958811)
+      (xy -3.083537 2.217173) (xy -2.866492 2.472412) (xy -2.671818 2.671886) (xy -2.127245 3.131612)
+      (xy -1.54339 3.470844) (xy -0.916452 3.691027) (xy -0.242632 3.793608) (xy 0.278165 3.795221)
+      (xy 0.96307 3.698113)) (layer B.SilkS) (width 0.01))
+  )
   (module ESProg:bsilk360 (layer B.Cu)
     (at 125.8 66.1)
@@
       (net 8 "Net-(S2-Pad1)") (solder_mask_margin 0.1016))
   )
+  (gr_text bit.ly/ouija8266 (at 127 96.5 180) (layer B.SilkS)
+    (effects (font (size 1 1) (thickness 0.15)) (justify mirror))
+  )
   (gr_text @glowascii (at 127.1 55 180) (layer B.SilkS)
